File: canfilter_g4.kicad_pcb (KiCad board)
At the start: 4 copper layers, 54.8 x 32.3 mm, 84 parts, among them J101 CAN1, J102 CAN2, J103 CAN3, J104 Vin, J105 Gnd, J106 SWD, J601 USB_C_Receptacle_USB2.0, Q101 AO3401A, SW101 BOOT0, U101 LP2985-3.3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

Commit message: QR code
Parts:
- added G***: LOGO, github_qrcode:github_qrcode, B.Cu at (141.8, 97.7)
