File: canfilter_g4.kicad_sch (KiCad schematic)
At the start: 47 parts, among them J101 CAN1, J102 CAN2, J103 CAN3, J104 Vin, J105 Gnd, J106 SWD, Q101 AO3401A, SW101 BOOT0, U101 LP2985-3.3, U102 STM32G474CBTx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

Commit message: QR code
Changed lines of the file:
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@@
+	)
+	(symbol
+		(lib_id "github_qrcode:LOGO")
+		(at 275.59 173.99 0)
+		(unit 1)
+		(exclude_from_sim no)
+		(in_bom yes)
+		(on_board yes)
+		(dnp no)
+		(fields_autoplaced yes)
+		(property "Reference" "#G101"
+			(at 275.59 165.227 0)
+			(effects
+				(font
+					(size 1.27 1.27)
+				)
+				(hide yes)
+			)
+		)
+		(property "Value" "LOGO"
+			(at 275.59 182.753 0)
+			(effects
+				(font
+					(size 1.27 1.27)
+				)
+				(hide yes)
+			)
+		)
+		(property "Footprint" ""
+			(at 275.59 173.99 0)
+			(effects
+				(font
+					(size 1.27 1.27)
+				)
+				(hide yes)
+			)
+		)
+		(property "Datasheet" ""
+			(at 275.59 173.99 0)
+			(effects
+				(font
+					(size 1.27 1.27)
+				)
+				(hide yes)
+			)
+		)
+		(property "Description" ""
+			(at 275.59 173.99 0)
+			(effects
+				(font
+					(size 1.27 1.27)
+				)
+				(hide yes)
+			)
+		)
+		(instances
+			(project ""
+				(path "/4f94f0b8-8c11-4faa-81ee-d093b0c859ad"
+					(reference "#G101")
+					(unit 1)
+				)
+			)
+		)
 	)
 	(symbol
