File: canfilter_g4.kicad_sch (KiCad schematic)
At the start: 47 parts, among them J101 CAN1, J102 CAN2, J103 CAN3, J104 Vin, J105 Gnd, J106 SWD, Q101 AO3401A, SW101 BOOT0, U101 LP2985-3.3, U102 STM32G474CBTx, Y101 8Mhz

Commit message: Project update
Parts:
- H101, H102, H103, H104, LOGO101: value ~ -> (none)
